Commit message: Fixed some more bugs

File: custom_ur_description/urdf/ur5e_joint_limited_robot.urdf.xacro (robot description, xacro)
@@ -28,7 +28,7 @@
   <link name="box_link">
     <visual>
-      <origin xyz="0.4 0.4 -0.5" rpy="0 0 0"/>
+      <origin xyz="0 0 -0.5" rpy="0 0 0"/>
       <geometry>
-        <box size="1 1 1" />
+        <box size="3 3 1" />
       </geometry>
       <material name="box_yellow">
@@ -37,7 +37,7 @@
     </visual>
     <collision>
-      <origin xyz="0.4 0.4 -0.5" rpy="0 0 0"/>
+      <origin xyz="0 0 -0.5" rpy="0 0 0"/>
       <geometry>
-        <box size="1 1 1" />
+        <box size="3 3 1" />
       </geometry>
     </collision>

File: custom_ur_description/urdf/ur5e_robot.urdf.xacro (robot description, xacro)
@@ -21,7 +21,7 @@
   <link name="box_link">
     <visual>
-      <origin xyz="0.4 0.4 -0.5" rpy="0 0 0"/>
+      <origin xyz="0 0 -0.5" rpy="0 0 0"/>
       <geometry>
-        <box size="1 1 1" />
+        <box size="3 3 1" />
       </geometry>
       <material name="box_yellow">
@@ -30,7 +30,7 @@
     </visual>
     <collision>
-      <origin xyz="0.4 0.4 -0.5" rpy="0 0 0"/>
+      <origin xyz="0 0 -0.5" rpy="0 0 0"/>
       <geometry>
-        <box size="1 1 1" />
+        <box size="3 3 1" />
       </geometry>
     </collision>

Commit message: Added cylinder to robot URDF to avoid MoveIt self-collision

File: custom_ur_description/urdf/ur5e_joint_limited_robot.urdf.xacro (robot description, xacro)
@@ -5,5 +5,5 @@
   <xacro:include filename="$(find ur_e_description)/urdf/common.gazebo.xacro" />
   <!-- ur5e -->
-  <xacro:include filename="$(find ur_e_description)/urdf/ur5e.urdf.xacro" />
+  <xacro:include filename="$(find custom_ur_description)/urdf/ur5e.urdf.xacro" />
   <!-- arm -->
   <xacro:ur5e_robot prefix="" joint_limited="true"
@@ -26,9 +26,11 @@
     <origin xyz="0.0 0.0 0.0" rpy="0.0 0.0 0.0" />
   </joint>
+  <xacro:property name="box_size" value="3 3 1" />
+  <xacro:property name="box_translation" value="0 0 -0.5" />
   <link name="box_link">
     <visual>
-      <origin xyz="0 0 -0.5" rpy="0 0 0"/>
+      <origin xyz="${box_translation}" rpy="0 0 0"/>
       <geometry>
-        <box size="3 3 1" />
+        <box size="${box_size}" />
       </geometry>
       <material name="box_yellow">
@@ -37,7 +39,33 @@
     </visual>
     <collision>
-      <origin xyz="0 0 -0.5" rpy="0 0 0"/>
+      <origin xyz="${box_translation}" rpy="0 0 0"/>
       <geometry>
-        <box size="3 3 1" />
+        <box size="${box_size}" />
+      </geometry>
+    </collision>
+  </link>
+  <joint name="ee_cylinder_joint" type="fixed">
+    <parent link="tool0" />
+    <child link="ee_cylinder_link" />
+    <origin xyz="0.0 0.0 0.0" rpy="0.0 0.0 0.0" />
+  </joint>
+  <xacro:property name="cylinder_radius" value="0.06" />
+  <xacro:property name="cylinder_length" value="0.18" />
+  <xacro:property name="cylinder_translation" value="0 0 ${cylinder_length/2}" />
+  <xacro:property name="cylinder_rotation" value="0 0 ${pi/2}" />
+  <link name="ee_cylinder_link">
+    <visual>
+      <origin xyz="${cylinder_translation}" rpy="${cylinder_rotation}"/>
+      <geometry>
+        <cylinder radius="${cylinder_radius}" length="${cylinder_length}" />
+      </geometry>
+      <material name="cylinder_color">
+        <color rgba="0 0 0 1"/>
+      </material>
+    </visual>
+    <collision>
+      <origin xyz="${cylinder_translation}" rpy="${cylinder_rotation}"/>
+      <geometry>
+        <cylinder radius="${cylinder_radius}" length="${cylinder_length}" />
       </geometry>
     </collision>

File: custom_ur_description/urdf/ur5e_robot.urdf.xacro (robot description, xacro)
@@ -19,9 +19,11 @@
     <origin xyz="0.0 0.0 0.0" rpy="0.0 0.0 0.0" />
   </joint>
+  <xacro:property name="box_size" value="3 3 1" />
+  <xacro:property name="box_translation" value="0 0 -0.5" />
   <link name="box_link">
     <visual>
-      <origin xyz="0 0 -0.5" rpy="0 0 0"/>
+      <origin xyz="${box_translation}" rpy="0 0 0"/>
       <geometry>
-        <box size="3 3 1" />
+        <box size="${box_size}" />
       </geometry>
       <material name="box_yellow">
@@ -30,7 +32,33 @@
     </visual>
     <collision>
-      <origin xyz="0 0 -0.5" rpy="0 0 0"/>
+      <origin xyz="${box_translation}" rpy="0 0 0"/>
       <geometry>
-        <box size="3 3 1" />
+        <box size="${box_size}" />
+      </geometry>
+    </collision>
+  </link>
+  <joint name="ee_cylinder_joint" type="fixed">
+    <parent link="tool0" />
+    <child link="ee_cylinder_link" />
+    <origin xyz="0.0 0.0 0.0" rpy="0.0 0.0 0.0" />
+  </joint>
+  <xacro:property name="cylinder_radius" value="0.06" />
+  <xacro:property name="cylinder_length" value="0.18" />
+  <xacro:property name="cylinder_translation" value="0 0 ${cylinder_length/2}" />
+  <xacro:property name="cylinder_rotation" value="0 0 ${pi/2}" />
+  <link name="ee_cylinder_link">
+    <visual>
+      <origin xyz="${cylinder_translation}" rpy="${cylinder_rotation}"/>
+      <geometry>
+        <cylinder radius="${cylinder_radius}" length="${cylinder_length}" />
+      </geometry>
+      <material name="cylinder_color">
+        <color rgba="0 0 0 1"/>
+      </material>
+    </visual>
+    <collision>
+      <origin xyz="${cylinder_translation}" rpy="${cylinder_rotation}"/>
+      <geometry>
+        <cylinder radius="${cylinder_radius}" length="${cylinder_length}" />
       </geometry>
     </collision>

Commit message: Improvements to HRI, general improvements and bugfixes

File: custom_ur_description/urdf/ur5e_joint_limited_robot.urdf.xacro (robot description, xacro)
@@ -51,5 +51,5 @@
   </joint>
   <xacro:property name="cylinder_radius" value="0.06" />
-  <xacro:property name="cylinder_length" value="0.18" />
+  <xacro:property name="cylinder_length" value="0.191" />
   <xacro:property name="cylinder_translation" value="0 0 ${cylinder_length/2}" />
   <xacro:property name="cylinder_rotation" value="0 0 ${pi/2}" />

File: custom_ur_description/urdf/ur5e_robot.urdf.xacro (robot description, xacro)
@@ -44,5 +44,5 @@
   </joint>
   <xacro:property name="cylinder_radius" value="0.06" />
-  <xacro:property name="cylinder_length" value="0.18" />
+  <xacro:property name="cylinder_length" value="0.191" />
   <xacro:property name="cylinder_translation" value="0 0 ${cylinder_length/2}" />
   <xacro:property name="cylinder_rotation" value="0 0 ${pi/2}" />

Commit message: Changed urdf to avoid self-collision in webots

File: custom_ur_description/urdf/ur5e_joint_limited_robot.urdf.xacro (robot description, xacro)
@@ -18,5 +18,5 @@
   <joint name="world_joint" type="fixed">
     <parent link="world" />
-    <child link = "base_link" />
+    <child link="base_link" />
     <origin xyz="0.0 0.0 0.0" rpy="0.0 0.0 0.0" />
   </joint>
@@ -27,5 +27,5 @@
   </joint>
   <xacro:property name="box_size" value="3 3 1" />
-  <xacro:property name="box_translation" value="0 0 -0.5" />
+  <xacro:property name="box_translation" value="0 0 -0.55" />
   <link name="box_link">
     <visual>
@@ -51,5 +51,5 @@
   </joint>
   <xacro:property name="cylinder_radius" value="0.06" />
-  <xacro:property name="cylinder_length" value="0.191" />
+  <xacro:property name="cylinder_length" value="0.2" />
   <xacro:property name="cylinder_translation" value="0 0 ${cylinder_length/2}" />
   <xacro:property name="cylinder_rotation" value="0 0 ${pi/2}" />

File: custom_ur_description/urdf/ur5e_robot.urdf.xacro (robot description, xacro)
@@ -20,5 +20,5 @@
   </joint>
   <xacro:property name="box_size" value="3 3 1" />
-  <xacro:property name="box_translation" value="0 0 -0.5" />
+  <xacro:property name="box_translation" value="0 0 -0.55" />
   <link name="box_link">
     <visual>
@@ -44,5 +44,5 @@
   </joint>
   <xacro:property name="cylinder_radius" value="0.06" />
-  <xacro:property name="cylinder_length" value="0.191" />
+  <xacro:property name="cylinder_length" value="0.2" />
   <xacro:property name="cylinder_translation" value="0 0 ${cylinder_length/2}" />
   <xacro:property name="cylinder_rotation" value="0 0 ${pi/2}" />
